File: KiCad/CherryZXKeyboard.kicad_pcb (KiCad board)
At the start: 2 copper layers, 290 x 120 mm, 100 parts, among them J1 Conn_01x05_Female, J2 Conn_01x08_Female, SW1 1, SW10 E, SW11 D, SW12 X, SW13 4, SW14 R, SW15 F, SW16 C, SW17 5, SW18 T, SW19 G, SW2 Q, SW20 V, SW21 6, SW22 Y, SW23 H, SW24 B, SW25 7, SW26 U, SW27 J, SW28 N, SW29 8, SW3 A, SW30 I, SW31 K, SW32 M, SW33 9, SW34 O, SW35 L, SW36 SYM, SW37 0, SW38 P, SW39 ENT, SW4 CAP, SW40 SPC, SW41 CAP, SW42 ;, SW43 ", SW44 ,, SW45 SYM, SW46 BREAK, SW47 EXTEND, SW48 DOT, SW49 LEFT, SW5 2, SW50 INV VID, SW51 TRUE VID, SW52 CAPS LOCK, SW53 EDIT, SW54 DOWN, SW55 UP, SW56 RIGHT, SW57 GRAPH, SW58 DEL, SW6 W, SW7 S, SW8 Z, SW9 3, U1 4066, U2 4066, U3 4066, U4 4066, U5 4066

Commit message: New files
Parts:
- added REF**: SW_Cherry_MX_1.00u_PCB, Button_Switch_Keyboard:SW_Cherry_MX_1.00u_PCB, F.Cu at (321.7, 154.1)
- added REF**: SW_Cherry_MX_1.00u_PCB, Button_Switch_Keyboard:SW_Cherry_MX_1.00u_PCB, F.Cu at (83.7, 174.1)
- added REF**: SW_Cherry_MX_1.00u_PCB, Button_Switch_Keyboard:SW_Cherry_MX_1.00u_PCB, F.Cu at (332.7, 134.1)
- added REF**: SW_Cherry_MX_1.00u_PCB, Button_Switch_Keyboard:SW_Cherry_MX_1.00u_PCB, F.Cu at (63.7, 154.1)
- moved SW37 32.0 mm to (295.7, 94.1)
- moved SW34 32.0 mm to (270.8, 114.2)
- moved SW39 9.48 mm to (313.7, 134.1)
- moved SW41 9.48 mm to (302.7, 154.1)
- moved SW4 9.48 mm to (82.7, 154.1)
- moved SW45 9.48 mm to (102.7, 174.1)
- moved SW30 0.07 mm to (250.7, 114.2)
Connections:
- D4 pad 2: Net-(D4-Pad2) -> Net-(SW50-Pad2)
- RN1 pad 2: Net-(D4-Pad2) -> Net-(SW50-Pad2)
- RN4 pad 4: Net-(RN4-Pad4) -> VDD
- SW50 pad 2: Net-(D10-Pad1) -> Net-(SW50-Pad2)
- SW54 pad 1: Net-(RN4-Pad4) -> VDD
- SW55 pad 1: Net-(RN4-Pad4) -> VDD
- SW56 pad 1: Net-(RN4-Pad4) -> VDD
- SW57 pad 1: Net-(RN4-Pad4) -> VDD
- SW58 pad 1: Net-(RN4-Pad4) -> VDD
- U1 pad 6: Net-(D4-Pad2) -> Net-(SW50-Pad2)
Routing:
- net Net-(RN4-Pad4): track 408.4 -> 0.00 mm, vias 1 -> 0
- net VDD: track 592.2 -> 984.8 mm, vias 2 -> 4
- net Net-(SW50-Pad2): track 0.00 -> 77.4 mm, vias 0 -> 1
- net Net-(D10-Pad1): track 312.5 -> 287.7 mm
- net Net-(D4-Pad2): track 24.4 -> 0.00 mm
- net Net-(D30-Pad2): track 588.8 -> 564.5 mm, vias 0 -> 1
- net Net-(D8-Pad2): track 546.7 -> 557.1 mm
- net Net-(D14-Pad1): track 160.8 -> 170.7 mm
- net Net-(D16-Pad1): track 204.6 -> 195.1 mm
- net Net-(D24-Pad2): track 149.2 -> 141.9 mm
- net Net-(D17-Pad1): track 531.3 -> 524.6 mm
- net Net-(D15-Pad1): track 472.0 -> 466.1 mm, vias 1 -> 2
- net Net-(D25-Pad2): track 217.5 -> 222.6 mm
- net Net-(D19-Pad2): track 324.7 -> 329.7 mm
- net Net-(D20-Pad2): track 335.1 -> 340.0 mm
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