File: KiCad/CherryZXKeyboard.kicad_sch (KiCad schematic)
At the start: 100 parts, among them J1 Conn_01x05_Female, J2 Conn_01x08_Female, SW1 1, SW10 E, SW11 D, SW12 X, SW13 4, SW14 R, SW15 F, SW16 C, SW17 5, SW18 T, SW19 G, SW2 Q, SW20 V, SW21 6, SW22 Y, SW23 H, SW24 B, SW25 7, SW26 U, SW27 J, SW28 N, SW29 8, SW3 A, SW30 I, SW31 K, SW32 M, SW33 9, SW34 O, SW35 L, SW36 SYM, SW37 0, SW38 P, SW39 ENT, SW4 CAP, SW40 SPC, SW41 CAP, SW42 ;, SW43 ", SW44 ,, SW45 SYM, SW46 BREAK, SW47 EXTEND, SW48 DOT, SW49 LEFT, SW5 2, SW50 INV VID, SW51 TRUE VID, SW52 CAPS LOCK, SW53 EDIT, SW54 DOWN, SW55 UP, SW56 RIGHT, SW57 GRAPH, SW58 DEL, SW6 W, SW7 S, SW8 Z, SW9 3, U1 4066, U2 4066, U3 4066, U4 4066, U5 4066

Commit message: New files
Connections:
- net VDD: now also RN4.4 (R3), SW54.1, SW55.1, SW56.1, SW57.1, SW58.1
- net at D10.1 (K), J2.1 (Pin_1), SW1.2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: no longer SW50.2
- net at D4.2 (A), RN1.2 (R1), U1.6: now also SW50.2
Changed lines of the file:
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@@
   (junction (at 158.75 140.97) (diameter 0) (color 0 0 0 0)
   )
+  (junction (at 393.7 50.8) (diameter 0) (color 0 0 0 0)
+  )
   (junction (at 123.19 64.77) (diameter 0) (color 0 0 0 0)
   )
@@
   (junction (at 35.56 35.56) (diameter 0) (color 0 0 0 0)
   )
-  (junction (at 91.44 109.22) (diameter 0) (color 0 0 0 0)
-  )
   (junction (at 339.09 187.96) (diameter 0) (color 0 0 0 0)
   )
@@
   (junction (at 262.89 125.73) (diameter 0) (color 0 0 0 0)
   )
+  (junction (at 99.06 116.84) (diameter 0) (color 0 0 0 0)
+  )
   (junction (at 250.19 119.38) (diameter 0) (color 0 0 0 0)
   )
@@
     (stroke (width 0) (type default) (color 0 0 0 0))
   )
-  (wire (pts (xy 66.04 96.52) (xy 71.12 96.52))
+  (wire (pts (xy 66.04 97.79) (xy 71.12 97.79))
     (stroke (width 0) (type default) (color 0 0 0 0))
   )
@@
     (stroke (width 0) (type default) (color 0 0 0 0))
   )
-  (wire (pts (xy 91.44 120.65) (xy 91.44 109.22))
+  (wire (pts (xy 91.44 105.41) (xy 91.44 120.65))
     (stroke (width 0) (type default) (color 0 0 0 0))
   )
@@
     (stroke (width 0) (type default) (color 0 0 0 0))
   )
-  (wire (pts (xy 91.44 109.22) (xy 39.37 109.22))
-    (stroke (width 0) (type default) (color 0 0 0 0))
-  )
   (wire (pts (xy 143.51 173.99) (xy 143.51 203.2))
     (stroke (width 0) (type default) (color 0 0 0 0))
@@
     (stroke (width 0) (type default) (color 0 0 0 0))
   )
-  (wire (pts (xy 39.37 109.22) (xy 39.37 99.06))
+  (wire (pts (xy 39.37 99.06) (xy 39.37 116.84))
     (stroke (width 0) (type default) (color 0 0 0 0))
   )
@@
     (stroke (width 0) (type default) (color 0 0 0 0))
   )
+  (wire (pts (xy 393.7 33.02) (xy 393.7 50.8))
+    (stroke (width 0) (type default) (color 0 0 0 0))
+  )
   (wire (pts (xy 262.89 125.73) (xy 262.89 139.7))
     (stroke (width 0) (type default) (color 0 0 0 0))
@@
     (stroke (width 0) (type default) (color 0 0 0 0))
   )
-  (wire (pts (xy 71.12 96.52) (xy 71.12 97.79))
-    (stroke (width 0) (type default) (color 0 0 0 0))
-  )
   (wire (pts (xy 256.54 77.47) (xy 256.54 80.01))
     (stroke (width 0) (type default) (color 0 0 0 0))
@@
     (stroke (width 0) (type default) (color 0 0 0 0))
   )
-  (wire (pts (xy 91.44 109.22) (xy 91.44 105.41))
-    (stroke (width 0) (type default) (color 0 0 0 0))
-  )
   (wire (pts (xy 158.75 203.2) (xy 158.75 200.66))
     (stroke (width 0) (type default) (color 0 0 0 0))
@@
     (stroke (width 0) (type default) (color 0 0 0 0))
   )
-  (wire (pts (xy 66.04 127) (xy 66.04 96.52))
+  (wire (pts (xy 66.04 127) (xy 66.04 97.79))
     (stroke (width 0) (type default) (color 0 0 0 0))
   )
@@
     (stroke (width 0) (type default) (color 0 0 0 0))
   )
+  (wire (pts (xy 99.06 116.84) (xy 99.06 134.62))
+    (stroke (width 0) (type default) (color 0 0 0 0))
+  )
   (wire (pts (xy 220.98 160.02) (xy 213.36 160.02))
     (stroke (width 0) (type default) (color 0 0 0 0))
@@
     (stroke (width 0) (type default) (color 0 0 0 0))
   )
+  (wire (pts (xy 39.37 116.84) (xy 99.06 116.84))
+    (stroke (width 0) (type default) (color 0 0 0 0))
+  )
   (wire (pts (xy 118.11 64.77) (xy 123.19 64.77))
     (stroke (width 0) (type default) (color 0 0 0 0))
@@
     (stroke (width 0) (type default) (color 0 0 0 0))
   )
-  (wire (pts (xy 99.06 113.03) (xy 99.06 134.62))
+  (wire (pts (xy 99.06 113.03) (xy 99.06 116.84))
     (stroke (width 0) (type default) (color 0 0 0 0))
   )
@@
     (pin "2")
   )
+  (symbol (lib_id "power:VDD") (at 393.7 33.02 0) (unit 1)
+    (in_bom yes) (on_board yes)
+    (property "Reference" "#PWR0109" (id 0) (at 393.7 36.83 0)
+      (effects (font (size 1.27 1.27)) hide)
+    )
+    (property "Value" "VDD" (id 1) (at 394.081 29.7942 90)
+      (effects (font (size 1.27 1.27)) (justify left))
+    )
+    (property "Footprint" "" (id 2) (at 393.7 33.02 0)
+      (effects (font (size 1.27 1.27)) hide)
+    )
+    (property "Datasheet" "" (id 3) (at 393.7 33.02 0)
+      (effects (font (size 1.27 1.27)) hide)
+    )
+    (pin "1")
+  )
   (sheet_instances
     (path "/" (page "1"))
@@
       (reference "#PWR0108") (unit 1) (value "VSS") (footprint "")
     )
+    (path "/e9f37295-704e-4fca-8e6d-6a07cec612e8"
+      (reference "#PWR0109") (unit 1) (value "VDD") (footprint "")
+    )
     (path "/00000000-0000-0000-0000-0000649e400d"
